Commit message: Established communication with real dynamixel. 10sec data is collected to csv file

File: urdf/MX28AR.ros2_control.xacro (robot description, xacro)
@@ -6,9 +6,9 @@
         <plugin>dynamixel_hardware/DynamixelHardware</plugin>
         <param name="usb_port">/dev/ttyUSB0</param>
-        <param name="baud_rate">1000000</param>
-        <param name="use_dummy">true</param>
+        <param name="baud_rate">57600</param>
+        <!-- <param name="use_dummy">true</param> -->
       </hardware>
       <joint name="joint1">
-        <param name="id">11</param>
+        <param name="id">1</param>
         <command_interface name="position"/>
         <command_interface name="velocity"/>

File: urdf/MX28AR.xacro (robot description, xacro)
@@ -40,5 +40,5 @@
     <child link="link2"/>
     <origin xyz="0.0 -0.03 0.0" rpy="0 0 0"/>
-    <axis xyz="0 1 0"/>
+    <axis xyz="0 -1 0"/>
     <limit velocity="5.76" effort="2.5" lower="-${pi}" upper="${pi}" />
     <dynamics damping="0.2" friction="0.2"/>

Commit message: Corrected dynamixel performing trajectory according to real dynamixel. The trajectory in gazebo is performed nearly as good as in the real one

File: urdf/MX28AR.ros2_control.xacro (robot description, xacro)
@@ -7,9 +7,11 @@
         <param name="usb_port">/dev/ttyUSB0</param>
         <param name="baud_rate">57600</param>
-        <!-- <param name="use_dummy">true</param> -->
+        <param name="use_dummy">true</param>
       </hardware>
       <joint name="joint1">
         <param name="id">1</param>
         <command_interface name="position"/>
+                <param name="min">${-pi}</param>
+                <param name="max">${pi}</param>
         <command_interface name="velocity"/>
         <state_interface name="position"/>
@@ -17,4 +19,11 @@
         <state_interface name="effort"/>
       </joint>
+      <!-- <transmission name="transmissionjoint1">
+          <plugin>transmission_interface/SimpleTransmission</plugin>
+          <joint name="joint1" role="joint1">
+              <mechanical_reduction>193.0</mechanical_reduction>
+              <offset>0.0</offset>
+          </joint>
+      </transmission>       -->
     </ros2_control>
   </xacro:macro>

File: urdf/MX28AR.xacro (robot description, xacro)
@@ -46,5 +46,5 @@
   <gazebo reference="joint1">
       <implicitSpringDamper>true</implicitSpringDamper>
-      <springStiffness>6.0</springStiffness>
+      <springStiffness>1.0</springStiffness>
       <springReference>0.01</springReference>
       <stopErp>0.2</stopErp>
@@ -67,9 +67,9 @@
     </collision>
      <inertial>
-      <origin xyz="-3.0184870e-04 5.4043684e-04 0.047433464e-02" />
-      <mass value="9.8406837e-02" />
-      <inertia ixx="3.4543422e-05" ixy="-1.6031095e-08" ixz="-3.8375155e-07"
-               iyy="3.2689329e-05" iyz="2.8511935e-08"
-               izz="1.8850320e-05" />
+      <origin xyz="0 0 0" />
+      <mass value="0.003" />
+      <inertia ixx="0.0000003025" ixy="0.0" ixz="0.0"
+               iyy="0.0000003025" iyz="0.0"
+               izz="0.00000031" />
     </inertial>
   </link>
