Commit message: Added IMU on robotic leg attached to dynamixel -simulation working and rViz also but it isoreinted bad way

File: urdf/MX28AR.xacro (robot description, xacro)
@@ -1,6 +1,4 @@
-<?xml version="1.0"?>
-<robot xmlns:xacro="http://ros.org/wiki/xacro">
-<!-- Import Rviz colors -->
-<xacro:include filename="$(find one_dynamixel_simulation)/urdf/one_dynamixel_simulation.material.xacro" />
+<robot xmlns:ns0="http://ros.org/wiki/xacro">
+<ns0:include filename="$(find one_dynamixel_simulation)/urdf/one_dynamixel_simulation.material.xacro" />
   <joint name="origin_to_link1" type="fixed">
     <parent link="world" />
@@ -9,17 +7,16 @@
     <origin xyz="0 0 0.07" rpy="0 0 0" />
   </joint>
-  <!-- Link 1 -->
   <link name="link1">
     <visual>
-      <origin xyz="0 0 0" rpy="${pi/2} 0 0"/>
+      <origin xyz="0 0 0" rpy="${pi/2} 0 0" />
       <geometry>
-        <mesh filename="file://$(find one_dynamixel_simulation)/meshes/mx-28at_ar.stl" scale="0.001 0.001 0.001"/>
+        <mesh filename="file://$(find one_dynamixel_simulation)/meshes/mx-28at_ar.stl" scale="0.001 0.001 0.001" />
       </geometry>
-      <material name="grey"/>
+      <material name="grey" />
     </visual>
     <collision>
-      <origin xyz="0 0 0" rpy="${pi/2} 0 0"/>
+      <origin xyz="0 0 0" rpy="${pi/2} 0 0" />
       <geometry>
-        <mesh filename="file://$(find one_dynamixel_simulation)/meshes/mx-28at_ar.stl" scale="0.001 0.001 0.001"/>
+        <mesh filename="file://$(find one_dynamixel_simulation)/meshes/mx-28at_ar.stl" scale="0.001 0.001 0.001" />
       </geometry>
     </collision>
@@ -27,7 +24,5 @@
       <origin xyz="0.2407e-03 -12.903e-03 0.5949e-03" />
       <mass value="0.075" />
-      <inertia ixx="22649.62e-06" ixy="36.779e-06" ixz="-213.05e-06"
-               iyy="12868.3e-06" iyz="-1145.65e-06"
-               izz="17733.142e-06" />
+      <inertia ixx="22649.62e-06" ixy="36.779e-06" ixz="-213.05e-06" iyy="12868.3e-06" iyz="-1145.65e-06" izz="17733.142e-06" />
     </inertial>
   </link>
@@ -35,12 +30,11 @@
         <material>Gazebo/Grey</material>
   </gazebo>
-  <!-- Joint 1 -->
   <joint name="joint1" type="revolute">
-    <parent link="link1"/>
-    <child link="link2"/>
-    <origin xyz="0.0 -0.03 0.0" rpy="0 0 0"/>
-    <axis xyz="0 -1 0"/>
+    <parent link="link1" />
+    <child link="link2" />
+    <origin xyz="0.0 -0.03 0.0" rpy="0 0 0" />
+    <axis xyz="0 -1 0" />
     <limit velocity="5.76" effort="2.5" lower="-${pi}" upper="${pi}" />
-    <dynamics damping="0.2" friction="0.2"/>
+    <dynamics damping="0.2" friction="0.2" />
   </joint>
   <gazebo reference="joint1">
@@ -51,17 +45,16 @@
       <stopCfm>0.2</stopCfm>
   </gazebo>
-  <!--  Link 2 -->
   <link name="link2">
     <visual>
-      <origin xyz="0 0 0" rpy="${pi} 0 0"/>
+      <origin xyz="0 0 0" rpy="${pi} 0 0" />
       <geometry>
-        <mesh filename="file://$(find one_dynamixel_simulation)/meshes/hn07-n101.stl" scale="0.001 0.001 0.001"/>
+        <mesh filename="file://$(find one_dynamixel_simulation)/meshes/hn07-n101.stl" scale="0.001 0.001 0.001" />
       </geometry>
-      <material name="grey"/>
+      <material name="grey" />
     </visual>
     <collision>
-      <origin xyz="0 0 0" rpy="${pi} 0 0"/>
+      <origin xyz="0 0 0" rpy="${pi} 0 0" />
       <geometry>
-        <mesh filename="file://$(find one_dynamixel_simulation)/meshes/hn07-n101.stl" scale="0.001 0.001 0.001"/>
+        <mesh filename="file://$(find one_dynamixel_simulation)/meshes/hn07-n101.stl" scale="0.001 0.001 0.001" />
       </geometry>
     </collision>
@@ -69,7 +62,5 @@
       <origin xyz="0 0 0" />
       <mass value="0.003" />
-      <inertia ixx="0.0000003025" ixy="0.0" ixz="0.0"
-               iyy="0.0000003025" iyz="0.0"
-               izz="0.00000031" />
+      <inertia ixx="0.0000003025" ixy="0.0" ixz="0.0" iyy="0.0000003025" iyz="0.0" izz="0.00000031" />
     </inertial>
   </link>

Commit message: working optimization code

File: urdf/MX28AR.xacro (robot description, xacro)
@@ -36,10 +36,10 @@
     <axis xyz="0 -1 0" />
     <limit velocity="5.76" effort="2.5" lower="-${pi}" upper="${pi}" />
-    <dynamics damping="0.2" friction="0.2" />
+    <dynamics damping="0.2" friction="64.2" />
   </joint>
   <gazebo reference="joint1">
       <implicitSpringDamper>true</implicitSpringDamper>
       <springStiffness>1.0</springStiffness>
-      <springReference>0.01</springReference>
+      <springReference>64.01</springReference>
       <stopErp>0.2</stopErp>
       <stopCfm>0.2</stopCfm>

Commit message: working optimization, repaired colcon build message problem

File: urdf/MX28AR.xacro (robot description, xacro)
@@ -36,10 +36,10 @@
     <axis xyz="0 -1 0" />
     <limit velocity="5.76" effort="2.5" lower="-${pi}" upper="${pi}" />
-    <dynamics damping="0.2" friction="64.2" />
+    <dynamics damping="0.575" friction="0.538" />
   </joint>
   <gazebo reference="joint1">
       <implicitSpringDamper>true</implicitSpringDamper>
       <springStiffness>1.0</springStiffness>
-      <springReference>64.01</springReference>
+      <springReference>0.061</springReference>
       <stopErp>0.2</stopErp>
       <stopCfm>0.2</stopCfm>

Commit message: Added to optimization parameters StopCfm StopErp and PID values

File: urdf/MX28AR.xacro (robot description, xacro)
@@ -36,10 +36,10 @@
     <axis xyz="0 -1 0" />
     <limit velocity="5.76" effort="2.5" lower="-${pi}" upper="${pi}" />
-    <dynamics damping="0.575" friction="0.538" />
+    <dynamics damping="1.825" friction="1.288" />
   </joint>
   <gazebo reference="joint1">
       <implicitSpringDamper>true</implicitSpringDamper>
       <springStiffness>1.0</springStiffness>
-      <springReference>0.061</springReference>
+      <springReference>1.061</springReference>
       <stopErp>0.2</stopErp>
       <stopCfm>0.2</stopCfm>

Commit message: Added MX64AR optimization algorithm

File: urdf/MX28AR.xacro (robot description, xacro)
@@ -36,12 +36,12 @@
     <axis xyz="0 -1 0" />
     <limit velocity="5.76" effort="2.5" lower="-${pi}" upper="${pi}" />
-    <dynamics damping="1.825" friction="1.288" />
+    <dynamics damping="2.825" friction="2.788" />
   </joint>
   <gazebo reference="joint1">
       <implicitSpringDamper>true</implicitSpringDamper>
-      <springStiffness>1.0</springStiffness>
-      <springReference>1.061</springReference>
-      <stopErp>0.2</stopErp>
-      <stopCfm>0.2</stopCfm>
+      <springStiffness>0.5</springStiffness>
+      <springReference>0.061</springReference>
+      <stopErp>0.7</stopErp>
+      <stopCfm>0.45</stopCfm>
   </gazebo>
   <link name="link2">

File: urdf/MX64AR.xacro (robot description, xacro)
@@ -1,6 +1,4 @@
-<?xml version="1.0"?>
-<robot xmlns:xacro="http://ros.org/wiki/xacro">
-<!-- Import Rviz colors -->
-<xacro:include filename="$(find one_dynamixel_simulation)/urdf/one_dynamixel_simulation.material.xacro" />
+<robot xmlns:ns0="http://ros.org/wiki/xacro">
+<ns0:include filename="$(find one_dynamixel_simulation)/urdf/one_dynamixel_simulation.material.xacro" />
   <joint name="origin_to_link1" type="fixed">
     <parent link="world" />
@@ -9,17 +7,16 @@
     <origin xyz="0 0 0.07" rpy="0 0 0" />
   </joint>
-  <!-- Link 1 -->
   <link name="link1">
     <visual>
-      <origin xyz="0 0 0" rpy="${pi/2} 0 0"/>
+      <origin xyz="0 0 0" rpy="${pi/2} 0 0" />
       <geometry>
-        <mesh filename="file://$(find one_dynamixel_simulation)/meshes/mx-64at_ar.stl" scale="0.001 0.001 0.001"/>
+        <mesh filename="file://$(find one_dynamixel_simulation)/meshes/mx-64at_ar.stl" scale="0.001 0.001 0.001" />
       </geometry>
-      <material name="grey"/>
+      <material name="grey" />
     </visual>
     <collision>
-      <origin xyz="0 0 0" rpy="${pi/2} 0 0"/>
+      <origin xyz="0 0 0" rpy="${pi/2} 0 0" />
       <geometry>
-        <mesh filename="file://$(find one_dynamixel_simulation)/meshes/mx-64at_ar.stl" scale="0.001 0.001 0.001"/>
+        <mesh filename="file://$(find one_dynamixel_simulation)/meshes/mx-64at_ar.stl" scale="0.001 0.001 0.001" />
       </geometry>
     </collision>
@@ -27,7 +24,5 @@
       <origin xyz="0.1583e-03 -17.0242e-03 1.6784e-03" />
       <mass value="0.1295" />
-      <inertia ixx="56457.58e-06" ixy="-652.34e-06" ixz="646.99e-06"
-               iyy="29325.73e-06" iyz="-5892.95e-06"
-               izz="45111.81e-06" />
+      <inertia ixx="56457.58e-06" ixy="-652.34e-06" ixz="646.99e-06" iyy="29325.73e-06" iyz="-5892.95e-06" izz="45111.81e-06" />
     </inertial>
   </link>
@@ -35,33 +30,31 @@
         <material>Gazebo/Grey</material>
   </gazebo>
-  <!-- Joint 1 -->
   <joint name="joint1" type="revolute">
-    <parent link="link1"/>
-    <child link="link2"/>
-    <origin xyz="0.0 -0.03 0.0" rpy="0 0 0"/>
-    <axis xyz="0 -1 0"/>
+    <parent link="link1" />
+    <child link="link2" />
+    <origin xyz="0.0 -0.03 0.0" rpy="0 0 0" />
+    <axis xyz="0 -1 0" />
     <limit velocity="6.597" effort="6.0" lower="-${pi}" upper="${pi}" />
-    <dynamics damping="0.2" friction="0.2"/>
+    <dynamics damping="1.45" friction="1.45" />
   </joint>
   <gazebo reference="joint1">
       <implicitSpringDamper>true</implicitSpringDamper>
-      <springStiffness>1.0</springStiffness>
+      <springStiffness>0.5</springStiffness>
       <springReference>0.01</springReference>
-      <stopErp>0.2</stopErp>
-      <stopCfm>0.2</stopCfm>
+      <stopErp>0.7</stopErp>
+      <stopCfm>0.45</stopCfm>
   </gazebo>
-  <!--  Link 2 -->
   <link name="link2">
     <visual>
-      <origin xyz="0 0 0" rpy="${pi} 0 0"/>
+      <origin xyz="0 0 0" rpy="${pi} 0 0" />
       <geometry>
-        <mesh filename="file://$(find one_dynamixel_simulation)/meshes/hn05_n102.stl" scale="0.001 0.001 0.001"/>
+        <mesh filename="file://$(find one_dynamixel_simulation)/meshes/hn05_n102.stl" scale="0.001 0.001 0.001" />
       </geometry>
-      <material name="grey"/>
+      <material name="grey" />
     </visual>
     <collision>
-      <origin xyz="0 0 0" rpy="${pi} 0 0"/>
+      <origin xyz="0 0 0" rpy="${pi} 0 0" />
       <geometry>
-        <mesh filename="file://$(find one_dynamixel_simulation)/meshes/hn05_n102.stl" scale="0.001 0.001 0.001"/>
+        <mesh filename="file://$(find one_dynamixel_simulation)/meshes/hn05_n102.stl" scale="0.001 0.001 0.001" />
       </geometry>
     </collision>
@@ -69,7 +62,5 @@
       <origin xyz="0 0 0" />
       <mass value="0.003" />
-      <inertia ixx="0.000000588" ixy="0.0" ixz="0.0"
-               iyy="0.0000002039" iyz="0.0"
-               izz="0.000000588" />
+      <inertia ixx="0.000000588" ixy="0.0" ixz="0.0" iyy="0.0000002039" iyz="0.0" izz="0.000000588" />
     </inertial>
   </link>
